File: pcb/rokibo_R/rokibo_R.kicad_sch (KiCad schematic)
At the start: 46 parts, among them SW100 SW_Push, SW101 SW_Push, SW102 SW_Push, SW103 SW_Push, SW104 SW_Push, SW105 SW_Push, SW106 SW_Push, SW107 SW_Push, SW108 SW_Push, SW109 SW_Push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

Commit message: fix: Use XIAO BLE footprint with hole
Parts:
- H100, H101, H102, H103, H104, H105: value (none) -> ~
- U100: footprint rokibo:XIAO_nRF52840_wBAT_wNFC -> rokibo:XIAO_nRF52840_wBAT_wNFC_1
Changed lines of the file:
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@@
 			)
 		)
-		(property "Value" ""
+		(property "Value" "~"
 			(at 196.85 128.2699 0)
 			(effects
@@
 			)
 		)
-		(property "Value" ""
+		(property "Value" "~"
 			(at 222.25 128.2699 0)
 			(effects
@@
 			)
 		)
-		(property "Value" ""
+		(property "Value" "~"
 			(at 171.45 128.2699 0)
 			(effects
@@
 			)
 		)
-		(property "Footprint" "rokibo:XIAO_nRF52840_wBAT_wNFC"
+		(property "Footprint" "rokibo:XIAO_nRF52840_wBAT_wNFC_1"
 			(at 43.18 29.21 0)
 			(effects
@@
 			)
 		)
-		(property "Value" ""
+		(property "Value" "~"
 			(at 158.75 128.2699 0)
 			(effects
@@
 			)
 		)
-		(property "Value" ""
+		(property "Value" "~"
 			(at 209.55 128.2699 0)
 			(effects
@@
 			)
 		)
-		(property "Value" ""
+		(property "Value" "~"
 			(at 184.15 128.2699 0)
 			(effects

Commit message: fix: Update tracks
Connections:
- net CS: now also U100.16 (NFC2_0.10); no longer U100.7 (P1.11_D6_TX)
- net MOTION: now also U100.6 (P0.05_A5_D5_SCL); no longer U100.15 (NFC1_0.09)
- net SCLK: now also U100.15 (NFC1_0.09); no longer U100.6 (P0.05_A5_D5_SCL)
- net SDIO: now also U100.7 (P1.11_D6_TX); no longer U100.16 (NFC2_0.10)
